Commit message: Fixed container

File: pycram/resources/robots/tiago_dual.urdf (robot description, URDF)
Before this commit: robot tiago_dual, 69 links, 68 joints
Joints:
- joint gripper_left_grasping_frame_joint: origin xyz=0 0 -0.12 rpy=-1.5708 1.5708 0 -> xyz=0 0 -0.15 rpy=-1.5708 1.5708 0
- joint gripper_right_grasping_frame_joint: origin xyz=0 0 -0.12 rpy=-1.5708 1.5708 0 -> xyz=0 0 -0.15 rpy=-1.5708 1.5708 0
